File: Electronics/Glue Board/Glue Board.kicad_pcb (KiCad board)
At the start: 4 copper layers, 81.3 x 52.8 mm, 87 parts, among them J1 Conn_01x02_Male, J2 Barrel_Jack, J3 Conn_01x02_Male, J4 Conn_02x06_Odd_Even, J5 Conn_01x02_Male, J6 Conn_01x05_Female, J7 Conn_01x04_Male, J8 Conn_02x03_Odd_Even, Q1 CSD17501Q5A, SW1 SW_SPST, SW2 SW_SPST, U1 PCA9685PW, U2 DRV8871DDA, U3 VNH5019ATR-E, U4 ADS1115IDGS, U5 NCP1117-5.0_SOT223, U6 TPS2121RUXR, U7 AMC1301DWVR, U8 INA260, U9 INA260

Commit message: Glue Board - Rev A - Production
Glue Board - Rev A - Production
Parts:
- U6: moved to F.Cu
- moved U9 23.7 mm to (217.7, 88.1), turned to 90 degrees
- moved C6 23.7 mm to (234.4, 89.7)
- moved U8 23.5 mm to (224.0, 88.1), turned to 90 degrees
- moved J7 17.1 mm to (205.2, 88.4)
- moved R40 16.8 mm to (215.6, 81.8), turned to 270 degrees
- moved R8 16.7 mm to (231.6, 70.6), turned to 90 degrees
- moved C9 16.5 mm to (221.2, 51.8), turned to 90 degrees
- moved J4 16.3 mm to (202.7, 68.1)
- moved R38 15.5 mm to (217.2, 81.8), turned to 270 degrees
- moved R9 14.5 mm to (202.9, 56.4), turned to 0 degrees
- moved C23 14.2 mm to (218.9, 81.8), turned to 90 degrees
- moved C22 13.9 mm to (225.3, 81.8), turned to 90 degrees
- moved D2 13.3 mm to (210.1, 61.5)
- moved R37 13.3 mm to (223.5, 81.8), turned to 270 degrees
- moved R39 13.2 mm to (222.0, 81.8), turned to 270 degrees
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Routing:
- net SCL: track 0.00 -> 120.8 mm, vias 0 -> 4
- net GND: track 0.00 -> 117.8 mm, vias 0 -> 46
- net SDA: track 0.00 -> 111.9 mm, vias 0 -> 4
- net +5V: track 0.00 -> 82.6 mm, vias 0 -> 12
- net OUTB: track 0.00 -> 73.3 mm, vias 0 -> 5
- net OUTA: track 0.00 -> 64.4 mm, vias 0 -> 3
- net VCC: track 0.00 -> 59.5 mm, vias 0 -> 9
- net Net-(C5-Pad1): track 0.00 -> 48.8 mm, vias 0 -> 4
- net VLOGIC_BAT: track 29.2 -> 76.6 mm, vias 0 -> 1
- net IN2: track 0.00 -> 45.1 mm
- net DRIVE_CS_ADC: track 0.00 -> 44.5 mm, vias 0 -> 2
- net IN1: track 0.00 -> 44.4 mm
- net Net-(C1-Pad1): track 0.00 -> 43.3 mm, vias 0 -> 3
- net INA: track 0.00 -> 42.2 mm, vias 0 -> 2
- net DRIVE_PWM: track 0.00 -> 36.6 mm, vias 0 -> 2
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- added copper zone on In2.Cu, net +5V
- added copper zone on In1.Cu, net GND
- added copper zone on F.Cu, net Net-(C7-Pad1)
- added copper zone on In2.Cu, net OUTA
- added copper zone on In2.Cu, net OUTB
- added copper zone on In2.Cu, net VBUS
- added copper zone on In2.Cu, net VCC
Other:
- outline, holes or cut-outs redrawn
- board text added: "BY: ARKO"
- board text added: "GLUE BOARD"
